File: Hardware/Schematic.sch (EAGLE design)
At the start: 103 parts, among them IC1 BQ25180YBGR_BQ25180YBGR, IC2 RT6160AWSC_RT6160AWSC, IC3 BMA423_BMA423, IC4 DRV2605YZFR, J1 TC2030-IDC_TC2030-IDC, J3 503480-2400, J4 KH-TYPE-C-16P, Q1 20V/4.2A/52mΩ/1.4W, Q3 ESP32_C6_LIBRARY_6_SI1308EDL-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, U3 MAX17048G+T10, X1 32MHz, X2 32.768kHz

Commit message: Add files via upload
Parts:
- removed TP3, TP6: HECTOR_WATCH_1_TPTP20R, InkTime_v5:HECTOR_WATCH_1_TPTP20R
- added TP_3V3, TP_3V3V, TP_GND, TP_VREG: HECTOR_WATCH_1_TPTP20R, InkTime_v5:HECTOR_WATCH_1_TPTP20R
- C9: value 820pF -> 820pF N.C.
- L5: value (none) -> 68uH
- renumbered TP4 to TP_RESET, U$1 to U1, U$2 to L5
Connections:
- removed net N$9: C18.2, U1.P0.01/XL2@F2, X2.1
- new net N$2: C18.2, U1.P0.01/XL2@F2, X2.2
- net 3V3/2.4A: now also TP_3V3.TP, TP_3V3V.TP; no longer TP_SWDCLK.TP
- net GND: now also TP_GND.TP; no longer TP6.TP
- net N$10: now also X2.1; no longer X2.2
- net SWDCLK: now also TP_SWDCLK.TP; no longer TP3.TP
- net VREG: now also TP_VREG.TP
Other:
- note added: "DEC3"
- note added: "DEC4_6"
- note added: "IMU"
- note added: "P0.00/XL1"
- note added: "P0.00/XL2"
- moved on the sheet: TP_ON, TP_SWDCLK
